File: Hardware/Rev.1/GameConsoleRev1/GameConsoleRev1.kicad_pcb (KiCad board)
At the start: 4 copper layers, 95 x 90.6 mm, 147 parts, among them J1 SWD-DAPLink, J10 Conn_01x40, J11 Conn_01x08_Pin, J12 Conn_01x08_Pin, J13 Micro_SD_Card, J14 Through Hole, J2 USB_C_Receptacle_USB2.0_14P, J3 L Channel, J4 R Channel, J5 JST, J6 Pack Temp, J7 HDMI_A, J8 Inputs, J9 Button Pulls, Q1 NMOS, Q2 NMOS, Q3 NTR1P02T1G, SW1 NRST, SW2 NRST, SW3 BOOTSEL, SW5 SW_SPDT, U1 RP2350B-QFN80, U10 PAM8302AAS, U11 PAM8302AAS, U2 BQ29700DSER, U3 BQ24073RGT, U4 AMS1117-3.3, U5 W25Q128JVS, U6 ESP-PSRAM64, U8 TLV61070ADBV, Y1 ABM8-272-T3 [12MHz]

Commit message: A
Parts:
- added C44: 10u, Capacitor_SMD:C_0402_1005Metric, F.Cu at (107.3, 45.0)
- added C45: 10u, Capacitor_SMD:C_0402_1005Metric, F.Cu at (172.7, 50.3)
- added C46: 10u, Capacitor_SMD:C_0402_1005Metric, F.Cu at (92.9, 97.3)
- added C47: 10u, Capacitor_SMD:C_0402_1005Metric, F.Cu at (179.9, 88.9)
- added D11: BLUE, LED_SMD:LED_0603_1608Metric, F.Cu at (132.1, 91.2)
- added D12: RED, LED_SMD:LED_0603_1608Metric, F.Cu at (148.2, 101.0)
- added D13: GREEN, LED_SMD:LED_0603_1608Metric, F.Cu at (151.2, 101.0)
- added D14: GREEN, LED_SMD:LED_0603_1608Metric, F.Cu at (154.1, 101.0)
- added D15: AMBER, LED_SMD:LED_0603_1608Metric, F.Cu at (157.1, 101.0)
- added D16: AMBER, LED_SMD:LED_0603_1608Metric, F.Cu at (160.0, 101.0)
- added D3: WS2812, LED_SMD:LED_WS2812_PLCC6_5.0x5.0mm_P1.6mm, F.Cu at (171.7, 46.0)
- added D4: WS2812, LED_SMD:LED_WS2812_PLCC6_5.0x5.0mm_P1.6mm, F.Cu at (103.0, 45.9)
- added D5: WS2812, LED_SMD:LED_WS2812_PLCC6_5.0x5.0mm_P1.6mm, F.Cu at (91.8, 93.1)
- added D6: WS2812, LED_SMD:LED_WS2812_PLCC6_5.0x5.0mm_P1.6mm, F.Cu at (180.6, 93.1)
- added J15: Conn_01x09_Pin, Connector_PinSocket_2.54mm:PinSocket_1x11_P2.54mm_Vertical, F.Cu at (175.1, 69.2)
- added R49: 1k, Resistor_SMD:R_0805_2012Metric, F.Cu at (132.3, 89.4)
- added R50: 1k, Resistor_SMD:R_0805_2012Metric, F.Cu at (148.2, 97.7)
- added R51: 1k, Resistor_SMD:R_0805_2012Metric, F.Cu at (151.2, 97.7)
- added R52: 1k, Resistor_SMD:R_0805_2012Metric, F.Cu at (154.1, 97.7)
- added R53: 1k, Resistor_SMD:R_0805_2012Metric, F.Cu at (157.1, 97.7)
- added R54: 1k, Resistor_SMD:R_0805_2012Metric, F.Cu at (160.0, 97.7)
- moved C2 2.70 mm to (144.8, 87.7)
Connections:
- net /RP2350B MCU/GPIO10 renamed /Power/GPIO10
- net /RP2350B MCU/GPIO12 renamed /Power/GPIO12
- net /RP2350B MCU/GPIO13 renamed /Power/GPIO13
- net /RP2350B MCU/GPIO14 renamed /Power/GPIO14
- net /RP2350B MCU/GPIO15 renamed /Power/GPIO15
- net /RP2350B MCU/GPIO16 renamed /Power/GPIO16
- net /RP2350B MCU/GPIO17 renamed /Power/GPIO17
- net /RP2350B MCU/GPIO18 renamed /Power/GPIO18
- net /RP2350B MCU/GPIO19 renamed /Power/GPIO19
- net /RP2350B MCU/GPIO2 renamed /Power/GPIO2
- net /RP2350B MCU/GPIO20 renamed /Power/GPIO20
- net /RP2350B MCU/GPIO21 renamed /Power/GPIO21
- net /RP2350B MCU/GPIO22 renamed /Power/GPIO22
- net /RP2350B MCU/GPIO23 renamed /Power/GPIO23
- net /RP2350B MCU/GPIO24 renamed /Power/GPIO24
- net /RP2350B MCU/GPIO25 renamed /Power/GPIO25
- net /RP2350B MCU/GPIO26 renamed /Power/GPIO26
- net /RP2350B MCU/GPIO27 renamed /Power/GPIO27
- net /RP2350B MCU/GPIO28 renamed /Power/GPIO28
- net /RP2350B MCU/GPIO29 renamed /Power/GPIO29
- net /RP2350B MCU/GPIO3 renamed /Power/GPIO3
- net /RP2350B MCU/GPIO32 renamed /Power/GPIO32
- net /RP2350B MCU/GPIO33 renamed /Power/GPIO33
- net /RP2350B MCU/GPIO35 renamed /Power/GPIO35
- net /RP2350B MCU/GPIO4 renamed /Power/GPIO4
- net /RP2350B MCU/GPIO40 renamed /Power/GPIO40
- net /RP2350B MCU/GPIO41 renamed /Power/GPIO41
- net /RP2350B MCU/GPIO42 renamed /Power/GPIO42
- net /RP2350B MCU/GPIO43 renamed /Power/GPIO43
- net /RP2350B MCU/GPIO44 renamed /Power/GPIO44
- net /RP2350B MCU/GPIO5 renamed /Power/GPIO5
- J13 pad 1: /RP2350B MCU/Peripherals/SD Card/DAT2 -> unconnected-(J13-DAT2-Pad1)
- J13 pad 5: /RP2350B MCU/Peripherals/SD Card/CLK -> /Power/GPIO34
- J13 pad 8: /RP2350B MCU/Peripherals/SD Card/DAT1 -> unconnected-(J13-DAT1-Pad8)
- U1 pad 3: /RP2350B MCU/GPIO6 -> /Power/GPIO6
- U1 pad 38: /RP2350B MCU/GPIO30 -> /Power/GPIO30
- U1 pad 39: /RP2350B MCU/GPIO31 -> /Power/GPIO31
- U1 pad 4: /RP2350B MCU/GPIO7 -> /Power/GPIO7
- U1 pad 43: /RP2350B MCU/GPIO34 -> /Power/GPIO34
- U1 pad 45: /RP2350B MCU/GPIO36 -> /Power/GPIO36
- U1 pad 46: /RP2350B MCU/GPIO37 -> /Power/GPIO37
- U1 pad 47: /RP2350B MCU/GPIO38 -> /Power/GPIO38
- U1 pad 48: /RP2350B MCU/GPIO39 -> /Power/GPIO39
- U1 pad 56: /RP2350B MCU/GPIO45 -> /Power/GPIO45
- U1 pad 57: /RP2350B MCU/GPIO46 -> /Power/GPIO46
- U1 pad 58: /RP2350B MCU/GPIO47 -> /Power/GPIO47
- U1 pad 7: /RP2350B MCU/GPIO9 -> /Power/GPIO9
- U1 pad 77: /RP2350B MCU/GPIO0 -> /Power/GPIO0
- U1 pad 78: /RP2350B MCU/GPIO1 -> /Power/GPIO1
- U1 pad 9: /RP2350B MCU/GPIO11 -> /Power/GPIO11
Routing:
- net Net-(D5-DOUT): track 0.00 -> 97.3 mm, vias 0 -> 2
- net +5V: track 267.3 -> 349.4 mm, vias 27 -> 28
- net Net-(D3-DOUT): track 0.00 -> 78.3 mm, vias 0 -> 2
- net /Power/GPIO47: track 17.2 -> 94.0 mm, vias 0 -> 2
- net /Power/GPIO37: track 0.00 -> 64.5 mm, vias 0 -> 3
- net /Power/GPIO6: track 0.00 -> 63.5 mm, vias 0 -> 3
- net /Power/GPIO31: track 0.00 -> 58.0 mm, vias 0 -> 2
- net Net-(D4-DOUT): track 0.00 -> 57.3 mm, vias 0 -> 2
- net /Power/GPIO9: track 0.00 -> 55.8 mm, vias 0 -> 2
- net /Power/GPIO36: track 0.00 -> 54.0 mm, vias 0 -> 2
- net /Power/GPIO39: track 0.00 -> 51.8 mm, vias 0 -> 2
- net /Power/GPIO11: track 0.00 -> 51.1 mm, vias 0 -> 2
- net /Power/GPIO46: track 0.00 -> 46.3 mm, vias 0 -> 2
- net /Power/GPIO30: track 0.00 -> 45.1 mm, vias 0 -> 1
- net /Power/GPIO34: track 0.00 -> 43.3 mm, vias 0 -> 2
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