File: Hardware/Rev.1/GameConsoleRev1/GameConsoleRev1.kicad_sch (KiCad schematic)
At the start: 0 parts

Commit message: Added sprites
Parts:
- added H1, H2, H3, H4: MountingHole, MountingHole:MountingHole_3.2mm_M3_Pad_Via, symbol Mechanical:MountingHole
Other:
- sheet Power ports: added USB_D+, USB_D-, {GPIO[0..47]}; removed none
- sheet RP2350B MCU ports: added USB_D+, USB_D-, {GPIO[0..47]}; removed none
